Commit message: Edited 3D files: adusing actual propeller model

File: blueboat_description/urdf/thrusters.xacro (robot description, xacro)
@@ -2,6 +2,6 @@
 <robot xmlns:xacro="http://www.ros.org/wiki/xacro">
   <!-- Propeller models from: https://github.com/markusbuchholz/gazebosim_blueboat_ardupilot_sitl/tree/main/SITL_Models/Gazebo/models/blueboat/meshes -->
-  <xacro:property name="prop_mesh_cw" value="package://blueboat_description/meshes/bluerov2_propcw.dae"/>
-  <xacro:property name="prop_mesh_ccw" value="package://blueboat_description/meshes/bluerov2_propccw.dae"/>
+  <xacro:property name="prop_mesh_cw" value="package://blueboat_description/meshes/BlueBoat_weedless_propeller_CW.dae"/>
+  <xacro:property name="prop_mesh_ccw" value="package://blueboat_description/meshes/BlueBoat_weedless_propeller_CCW.dae"/>
   <xacro:property name="prop_r" value="0.056"/>
   <xacro:property name="prop_l" value="0.035"/>
@@ -10,4 +10,5 @@
     <link name="${ns}/thruster${thruster_id}">
       <visual>
+        <origin xyz="0 0 0" rpy="0 0 ${pi}" />
         <geometry>
           <xacro:if value="${thruster_id in [1]}">
