Commit message: Added BlueBoat.dae and edited inertia matrix

File: blueboat_description/urdf/blueboat.xacro (robot description, xacro)
@@ -20,5 +20,5 @@
   <!-- Center of gravity -->
   <xacro:property name="z_cog" value="${-buoyant_correction*z_size}"/>
-  <xacro:property name="visual_mesh_file" value="package://blueboat_description/meshes/BlueBoat.stl"/>
+  <xacro:property name="visual_mesh_file" value="package://blueboat_description/meshes/BlueBoat.dae"/>
   <xacro:property name="collision_mesh_file" value="package://blueboat_description/meshes/BlueBoat.stl"/>
   <!-- Vehicle base link -->
@@ -28,8 +28,10 @@
         <origin xyz="0 0 ${z_cog}" rpy = "0 0 0"/>
     <!-- Inertia taken from: https://github.com/markusbuchholz/gazebosim_blueboat_ardupilot_sitl/blob/main/SITL_Models/Gazebo/models/blueboat/model.sdf-->
-        <inertia ixx="2.42369" ixy="0" ixz="0" iyy="3.9235025" iyz="0" izz="5.6403125"/>
+        <!-- <inertia ixx="2.42369" ixy="0" ixz="0" iyy="3.9235025" iyz="0" izz="5.6403125"/> -->
+    <!-- Inertia computed from .stl file-->
+        <inertia ixx="100.338" ixy="1.223" ixz="-3.53" iyy="70.777" iyz="1.188" izz="149.489"/>
     </inertial>
     <visual>
-        <origin xyz="0 0 ${z_cog}" rpy = "0 0 0"/>
+        <origin xyz="0 -0.01 ${z_cog+0.255}" rpy = "${pi/2} 0 0"/>
         <geometry>
         <mesh filename="${visual_mesh_file}"/>

Commit message: Minor changes

File: blueboat_description/urdf/blueboat.xacro (robot description, xacro)
@@ -8,12 +8,12 @@
   <xacro:property name="density" value="$(arg density)"/>
   <!-- Main body -->
-  <xacro:property name="x_size" value="0.40"/>
-  <xacro:property name="y_size" value="0.25"/>
-  <xacro:property name="z_size" value="0.1"/>
-  <xacro:property name="mass" value="14.8"/>
+  <xacro:property name="x_size" value="1.2"/>
+  <xacro:property name="y_size" value="0.91"/>
+  <xacro:property name="z_size" value="0.376"/>
+  <xacro:property name="mass" value="30.0"/>
   <!-- other props -->
   <xacro:property name="prop_mass" value="0.07"/>
   <!-- to set correct buoyancy volume with 1 % positive factor -->
-  <xacro:property name="buoyant_correction" value="${1.01*pow((mass + 6*prop_mass)/(density*x_size*y_size*z_size), 1./3)}"/>
+  <xacro:property name="buoyant_correction" value="${1.01*pow((mass + 2*prop_mass)/(density*x_size*y_size*z_size), 1./3)}"/>
   <!-- Center of buoyancy -->
   <xacro:property name="z_cob" value="${-buoyant_correction*z_size/4}"/>
@@ -26,12 +26,12 @@
     <inertial>
         <mass value="${mass}"/>
-        <origin xyz="0 0 ${z_cog}" rpy = "0 0 0"/>
-    <!-- Inertia taken from: https://github.com/markusbuchholz/gazebosim_blueboat_ardupilot_sitl/blob/main/SITL_Models/Gazebo/models/blueboat/model.sdf-->
-        <!-- <inertia ixx="2.42369" ixy="0" ixz="0" iyy="3.9235025" iyz="0" izz="5.6403125"/> -->
-    <!-- Inertia computed from .stl file-->
-        <inertia ixx="100.338" ixy="1.223" ixz="-3.53" iyy="70.777" iyz="1.188" izz="149.489"/>
+        <origin xyz="0 0 ${z_cog}" rpy = "${pi/2} 0 0"/>
+    <!-- Inertia computed from .stl file (likely incorrect)-->
+        <!-- <inertia ixx="100.338" ixy="1.223" ixz="-3.53" iyy="70.777" iyz="1.188" izz="149.489"/> -->
+    <!-- https://github.com/markusbuchholz/gazebosim_blueboat_ardupilot_sitl/blob/main/SITL_Models/Gazebo/models/blueboat/model.sdf -->
+        <inertia ixx="2.42369" ixy="0" ixz="0" iyy="3.9235025" iyz="0" izz="5.6403125"/>
     </inertial>
     <visual>
-        <origin xyz="0 -0.01 ${z_cog+0.255}" rpy = "${pi/2} 0 0"/>
+        <origin xyz="0 -0.01 ${z_cog+0.25}" rpy = "${pi/2} 0 0"/>
         <geometry>
         <mesh filename="${visual_mesh_file}"/>
@@ -42,5 +42,5 @@
     </visual>
     <collision>
-        <origin xyz="0 0 ${z_cob}"/>
+        <origin xyz="0 0 0"/>
         <!-- Box adjusted for buoyancy -->
         <geometry>

File: blueboat_description/urdf/hydrodynamics.xacro (robot description, xacro)
@@ -6,4 +6,6 @@
     <!-- Ignition notations from Handbook of Marine Craft, Fossen, 2011 -->
     <link_name>${ns}/base_link</link_name>
+    <!-- LIEVORE, MARCO. "Autonomous usv navigation and control for auv tracking via optimal,
+    collision-free trajectory generation." -->
     <!-- BlueROV2 heavy values from "6-DoF Modelling and Control of a Remotely Operated Vehicle"
         Wu, Master thesis, Flinder University, 2018  -->

File: blueboat_description/urdf/thrusters.xacro (robot description, xacro)
@@ -70,8 +70,8 @@
   <!-- all thrusters -->
   <xacro:thruster thruster_id="1">
-    <origin xyz="-0.488 -0.295 -0.01" rpy="0 0 0"/>
+    <origin xyz="-0.488 -0.295 -0.025" rpy="0 0 0"/>
   </xacro:thruster>
   <xacro:thruster thruster_id="2">
-    <origin xyz="-0.488 0.295 -0.01" rpy="0 0 0"/>
+    <origin xyz="-0.488 0.295 -0.025" rpy="0 0 0"/>
   </xacro:thruster>
 </robot>

Commit message: Large update, full robot interaction, controllers available for real robot.

File: blueboat_description/urdf/blueboat.xacro (robot description, xacro)
@@ -11,5 +11,5 @@
   <xacro:property name="y_size" value="0.91"/>
   <xacro:property name="z_size" value="0.376"/>
-  <xacro:property name="mass" value="30.0"/>
+  <xacro:property name="mass" value="16.01"/>
   <!-- other props -->
   <xacro:property name="prop_mass" value="0.07"/>
@@ -42,5 +42,5 @@
     </visual>
     <collision>
-        <origin xyz="0 0 0"/>
+        <origin xyz="0 0 0.05"/>
         <!-- Box adjusted for buoyancy -->
         <geometry>

File: blueboat_description/urdf/hydrodynamics.xacro (robot description, xacro)
@@ -6,6 +6,8 @@
     <!-- Ignition notations from Handbook of Marine Craft, Fossen, 2011 -->
     <link_name>${ns}/base_link</link_name>
+    <!-- BlueBoat Parameters -->
     <!-- LIEVORE, MARCO. "Autonomous usv navigation and control for auv tracking via optimal,
     collision-free trajectory generation." -->
+    <!-- BlueROV2 parameters -->
     <!-- M. von Benzon, F. F. Sørensen, E. Uth, J. Jouf-
     froy, J. Liniger, and S. Pedersen, “An open-source
@@ -13,47 +15,48 @@
     derwater robot,” Journal of Marine Science and
     Engineering, vol. 10, no. 12, p. 1898, 2022. -->
+    <!-- BlueROV2 -->
     <!-- Negative diagonal values of added mass matrix -->
-    <xDotU>-6.36</xDotU>
+    <xDotU>-5.5</xDotU>
+    <yDotV>-12.7</yDotV>
+    <zDotW>-14.57</zDotW>
+    <kDotP>-0.12</kDotP>z
+    <mDotQ>-0.12</mDotQ>
+    <nDotR>-0.12</nDotR>
+    <!-- Negative linear damping -->
+    <xU>-25.15</xU>
+    <yV>-7.364</yV>
+    <zW>-17.955</zW>
+    <kP>-10.888</kP>
+    <mQ>-20.761</mQ>
+    <nR>-3.744</nR>
+    <!-- Negative quadratic damping -->
+    <xUabsU>-33.800000000000004</xUabsU>
+    <yVabsV>-54.26875</yVabsV>
+    <zWabsW>-73.37135</zWabsW>
+    <kPabsP>-40.0</kPabsP>
+    <mQabsQ>-40.0</mQabsQ>
+    <nRabsR>-40.0</nRabsR>
+    <!-- BlueROV2 Heavy -->
+    <!-- Negative diagonal values of added mass matrix -->
+    <!-- <xDotU>-6.36</xDotU>
     <yDotV>-7.12</yDotV>
     <zDotW>-18.68</zDotW>
-    <kDotP>-0.189</kDotP>
+    <kDotP>-0.189</kDotP>z
     <mDotQ>-0.135</mDotQ>
-    <nDotR>-0.222</nDotR>
+    <nDotR>-0.222</nDotR> -->
     <!-- Negative linear damping -->
-    <xU>-29.34</xU>
-    <yV>-51.54</yV>
-    <zW>-17.955</zW>
+    <!-- <xU>-13.7</xU>
+    <yV>-0.</yV>
+    <zW>-33.</zW>
     <kP>-0.</kP>
     <mQ>-0.8</mQ>
-    <nR>-44.65</nR>
-    <!-- Negative quadratic damping [Fossen (6.62)] -->
-    <xUabsU>-141</xUabsU>
+    <nR>-0.</nR> -->
+    <!-- Negative quadratic damping -->
+    <!-- <xUabsU>-141</xUabsU>
     <yVabsV>-217</yVabsV>
     <zWabsW>-190</zWabsW>
     <kPabsP>-1.19</kPabsP>
     <mQabsQ>-0.47</mQabsQ>
-    <nRabsR>-1.5</nRabsR>
-    <!-- Previous values -->
-    <!-- Negative diagonal values of added mass matrix -->
-    <!-- <xDotU>-5.5</xDotU>
-    <yDotV>-12.7</yDotV>
-    <zDotW>-14.57</zDotW>
-    <kDotP>-0.12</kDotP>
-    <mDotQ>-0.12</mDotQ>
-    <nDotR>-0.12</nDotR> -->
-    <!-- Negative linear damping -->
-    <!-- <xU>-25.15</xU>
-    <yV>-7.364</yV>
-    <zW>-17.955</zW>
-    <kP>-10.888</kP>
-    <mQ>-20.761</mQ>
-    <nR>-3.744</nR> -->
-    <!-- Negative quadratic damping -->
-    <!-- <xUabsU>-33.800000000000004</xUabsU>
-    <yVabsV>-54.26875</yVabsV>
-    <zWabsW>-73.37135</zWabsW>
-    <kPabsP>-40.0</kPabsP>
-    <mQabsQ>-40.0</mQabsQ>
-    <nRabsR>-40.0</nRabsR> -->
+    <nRabsR>-1.9</nRabsR> -->
     </plugin>
 </gazebo>
